Commit message: Real-arm stack in Gazebo (virtual ESP) + fixes it uncovered
- arm_real_sim.launch.py + scripts/virtual_esp.py: the unchanged real-arm
  stack (RoverArmHardware, teleop, MoveIt) driving Gazebo through a virtual
  ESP32 (motor model, encoders, watchdog, failure drills). Gazebo's own
  controller manager runs in /gz with velocity joints; /clock bridged.
- Real arm: finger collision geometry now uses the finger meshes (the 9 cm
  spheres made every pose "in collision", so MoveIt could never plan);
  SRDF allows finger-finger contact.
- RoverArmHardware: closed loop now uses ff_gain as feed-forward
  (PWM = ff_gain*v + PI); ff_gain / pwm_deadband settable from the launch.
- RViz: wall-clock time and the real robot model for the real stack,
  world->stand_link TF, External Comm. on; teleop syncs RViz start/goal
  state when switching to AUTONOMOUS (fixes Plan starting from a stale pose).
- arm_real.launch.py: rviz and start_arm_py arguments. README updated.

Co-Authored-By: Claude Opus 5.5 <noreply@anthropic.com>

File: src/rover_arm_description/urdf/rover_arm_real.xacro (robot description, xacro)
@@ -5,4 +5,7 @@
        Set from the launch file: arm_real.launch.py open_loop_joints:=all -->
   <xacro:arg name="open_loop_joints" default="none"/>
+  <!-- Motor tuning, overridable from the launch file (arm_real.launch.py ff_gain:=... pwm_deadband:=...). -->
+  <xacro:arg name="ff_gain" default="100.0"/>
+  <xacro:arg name="pwm_deadband" default="0.0"/>
   <xacro:macro name="aluminum_material" params="link_name">
     <gazebo reference="${link_name}">
@@ -73,5 +76,5 @@
       <origin xyz="-0.013622 -0.083285 0" rpy="0 0 -3.141593" />
       <geometry>
-        <sphere radius="0.092785" />
+        <mesh filename="package://rover_arm_description/urdf/meshes/left_finger_link_collision.stl" />
       </geometry>
     </collision>
@@ -113,5 +116,5 @@
       <origin xyz="0.013622 -0.083285 0" rpy="3.141593 0 0" />
       <geometry>
-        <sphere radius="0.092785" />
+        <mesh filename="package://rover_arm_description/urdf/meshes/right_finger_link_collision.stl" />
       </geometry>
     </collision>
@@ -241,9 +244,10 @@
       <param name="ki">5.0</param>
       <param name="pwm_limit">255.0</param>
-      <!-- Open loop: PWM = ff_gain * motor velocity (rad/s). Tune on the bench. -->
-      <param name="ff_gain">100.0</param>
+      <!-- PWM per rad/s of motor velocity: the whole command in open loop, the feed-forward
+           in closed loop. Tune on the bench in open loop first. -->
+      <param name="ff_gain">$(arg ff_gain)</param>
       <!-- PWM below which the motors don't move. Small commands are scaled up past it
            while a motion is commanded. 0 = off; measure on the bench (open loop). -->
-      <param name="pwm_deadband">0.0</param>
+      <param name="pwm_deadband">$(arg pwm_deadband)</param>
       <param name="open_loop_joints">$(arg open_loop_joints)</param>
       <!-- Closed loop: motors get 0 PWM if /enc_angles is older than this. -->

File: src/rover_arm_description/urdf/rover_arm_sim.xacro (robot description, xacro)
@@ -2,4 +2,12 @@
 <robot xmlns:xacro="http://www.ros.org/wiki/xacro" name="rover_arm">
   <xacro:arg name="use_gazebo_ros2_control" default="true"/>
+  <!-- position (default, gazebo.launch.py) or velocity (arm_real_sim.launch.py: the
+       real-arm stack drives Gazebo through virtual_esp.py, which commands velocities). -->
+  <xacro:arg name="gz_command_interface" default="position"/>
+  <xacro:property name="gz_cmd_velocity" value="${'$(arg gz_command_interface)' == 'velocity'}"/>
+  <!-- Namespace + controller file for Gazebo's own controller manager. arm_real_sim
+       uses /gz so it doesn't clash with the real stack's /controller_manager. -->
+  <xacro:arg name="gz_namespace" default=""/>
+  <xacro:arg name="gz_controllers_file" default="ros2_controllers_sim.yaml"/>
   <xacro:macro name="aluminum_material" params="link_name">
     <gazebo reference="${link_name}">
@@ -326,56 +334,91 @@
     </hardware>
     <joint name="base_link_joint">
-      <command_interface name="position">
-        <param name="min">-1.570795</param>
-        <param name="max">1.570795</param>
-      </command_interface>
+      <xacro:if value="${gz_cmd_velocity}">
+        <command_interface name="velocity"/>
+      </xacro:if>
+      <xacro:unless value="${gz_cmd_velocity}">
+        <command_interface name="position">
+          <param name="min">-1.570795</param>
+          <param name="max">1.570795</param>
+        </command_interface>
+      </xacro:unless>
       <state_interface name="position"/>
       <state_interface name="velocity"/>
     </joint>
     <joint name="shoulder_link_joint">
-      <command_interface name="position">
-        <param name="min">-0.3927</param>
-        <param name="max">1.5708</param>
-      </command_interface>
+      <xacro:if value="${gz_cmd_velocity}">
+        <command_interface name="velocity"/>
+      </xacro:if>
+      <xacro:unless value="${gz_cmd_velocity}">
+        <command_interface name="position">
+          <param name="min">-0.3927</param>
+          <param name="max">1.5708</param>
+        </command_interface>
+      </xacro:unless>
       <state_interface name="position"/>
       <state_interface name="velocity"/>
     </joint>
     <joint name="elbow_link_joint">
-      <command_interface name="position">
-        <param name="min">-3.141593</param>
-        <param name="max">3.141593</param>
-      </command_interface>
+      <xacro:if value="${gz_cmd_velocity}">
+        <command_interface name="velocity"/>
+      </xacro:if>
+      <xacro:unless value="${gz_cmd_velocity}">
+        <command_interface name="position">
+          <param name="min">-3.141593</param>
+          <param name="max">3.141593</param>
+        </command_interface>
+      </xacro:unless>
       <state_interface name="position"/>
       <state_interface name="velocity"/>
     </joint>
     <joint name="wrist_link_joint">
-      <command_interface name="position">
-        <param name="min">-1.570795</param>
-        <param name="max">1.570795</param>
-      </command_interface>
+      <xacro:if value="${gz_cmd_velocity}">
+        <command_interface name="velocity"/>
+      </xacro:if>
+      <xacro:unless value="${gz_cmd_velocity}">
+        <command_interface name="position">
+          <param name="min">-1.570795</param>
+          <param name="max">1.570795</param>
+        </command_interface>
+      </xacro:unless>
       <state_interface name="position"/>
       <state_interface name="velocity"/>
     </joint>
     <joint name="palm_link_joint">
-      <command_interface name="position">
-        <param name="min">-3.141593</param>
-        <param name="max">3.141593</param>
-      </command_interface>
+      <xacro:if value="${gz_cmd_velocity}">
+        <command_interface name="velocity"/>
+      </xacro:if>
+      <xacro:unless value="${gz_cmd_velocity}">
+        <command_interface name="position">
+          <param name="min">-3.141593</param>
+          <param name="max">3.141593</param>
+        </command_interface>
+      </xacro:unless>
       <state_interface name="position"/>
       <state_interface name="velocity"/>
     </joint>
     <joint name="left_finger_link_joint">
-      <command_interface name="position">
-        <param name="min">-1.570795</param>
-        <param name="max">0.785398</param>
-      </command_interface>
+      <xacro:if value="${gz_cmd_velocity}">
+        <command_interface name="velocity"/>
+      </xacro:if>
+      <xacro:unless value="${gz_cmd_velocity}">
+        <command_interface name="position">
+          <param name="min">-1.570795</param>
+          <param name="max">0.785398</param>
+        </command_interface>
+      </xacro:unless>
       <state_interface name="position"/>
       <state_interface name="velocity"/>
     </joint>
     <joint name="right_finger_link_joint">
-      <command_interface name="position">
-        <param name="min">-0.785398</param>
-        <param name="max">1.570795</param>
-      </command_interface>
+      <xacro:if value="${gz_cmd_velocity}">
+        <command_interface name="velocity"/>
+      </xacro:if>
+      <xacro:unless value="${gz_cmd_velocity}">
+        <command_interface name="position">
+          <param name="min">-0.785398</param>
+          <param name="max">1.570795</param>
+        </command_interface>
+      </xacro:unless>
       <state_interface name="position"/>
       <state_interface name="velocity"/>
@@ -384,5 +427,8 @@
   <gazebo>
     <plugin filename="gz_ros2_control-system" name="gz_ros2_control::GazeboSimROS2ControlPlugin">
-      <parameters>$(find rover_arm_description)/config/ros2_controllers_sim.yaml</parameters>
+      <ros>
+        <namespace>$(arg gz_namespace)</namespace>
+      </ros>
+      <parameters>$(find rover_arm_description)/config/$(arg gz_controllers_file)</parameters>
     </plugin>
   </gazebo>
