Commit message: Terrain navigation sim: 3-marker ArUco run over hills and rocks
- rover_description: terrain_aruco.launch.py, generated terrain world
  (scripts/generate_terrain_world.py -> worlds/terrain_world.sdf,
  models/rover_terrain). Launch adds ground-truth 3D odometry (wheel
  odometry drifted ~80 deg per in-place turn), a ZED depth point cloud
  and speed caps for movement.py.
- rover_sim urdf/xacro: upstream front-right wheel rename and wheel
  limits (12 N·m, 15 rad/s); rocker friction 1000 (DART ignores mimic,
  chassis pitched ~45 deg); bogie limits +-30 deg (bogies flipped over).
- movement.py: turn in place with a dead band, stall back-up, ABORTED
  after 3 failed back-ups.
- goal_generator.py: publish the target ID before the goal so arrivals
  are reported for the right marker.

Tested in the GUI sim: all 3 markers reached in 69 s.

Co-Authored-By: Claude Opus 5.5 <noreply@anthropic.com>

File: src/rover_description/urdf/rover_raw.urdf (robot description, URDF)
Before this commit: robot rover_test_version, 13 links, 12 joints
Links:
- removed link left_back_wheel_link
- added link front_right_wheel_link, mass 3; collision cylinder length=0.184024 radius=0.119695; visual mesh filename=package://rover_description/urdf/meshes/front_right_wheel_l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
Joints:
- removed joint left_back_wheel_link_joint
- added joint front_right_wheel_link_joint: type continuous, parent right_bogie_link, child front_right_wheel_link, origin xyz=0.247131 -0.0135 -0.201737 rpy=0 0 0, axis 0 1 0, limit lower=0 upper=0 effort=12 velocity=15
- joint back_left_wheel_link_joint: limit lower=0 upper=0 effort=10 velocity=1 -> lower=0 upper=0 effort=12 velocity=15
- joint back_right_wheel_link_joint: limit lower=0 upper=0 effort=10 velocity=1 -> lower=0 upper=0 effort=12 velocity=15
- joint front_left_wheel_link_joint: limit lower=0 upper=0 effort=10 velocity=1 -> lower=0 upper=0 effort=12 velocity=15
- joint middle_left_wheel_link_joint: limit lower=0 upper=0 effort=10 velocity=1 -> lower=0 upper=0 effort=12 velocity=15
- joint middle_right_wheel_link_joint: limit lower=0 upper=0 effort=10 velocity=1 -> lower=0 upper=0 effort=12 velocity=15

File: src/rover_description/urdf/rover_raw.xacro (robot description, xacro)
@@ -90,14 +90,14 @@
     </collision>
   </link>
-  <link name="left_back_wheel_link">
-    <inertial>
-      <origin xyz="-0.000784 -0.092012 0.001876" rpy="1.570796 0 0" />
-      <mass value="3" />
-      <inertia ixx="0.019211" ixy="0" ixz="0" iyy="0.019211" iyz="0" izz="0.02149" />
-    </inertial>
-    <visual>
-      <origin xyz="-0.000784 -0.092012 0.001876" rpy="1.570796 0 0" />
-      <geometry>
-        <mesh filename="package://rover_description/urdf/meshes/left_back_wheel_link_visual.obj" />
+  <link name="front_right_wheel_link">
+    <inertial>
+      <origin xyz="-0.000784 -0.092012 0.001876" rpy="1.570796 0 0" />
+      <mass value="3" />
+      <inertia ixx="0.019211" ixy="0" ixz="0" iyy="0.019211" iyz="0" izz="0.02149" />
+    </inertial>
+    <visual>
+      <origin xyz="-0.000784 -0.092012 0.001876" rpy="1.570796 0 0" />
+      <geometry>
+        <mesh filename="package://rover_description/urdf/meshes/front_right_wheel_link_visual.obj" />
       </geometry>
     </visual>
@@ -252,5 +252,5 @@
     <child link="back_left_wheel_link" />
     <axis xyz="0 1 0" />
-    <limit effort="10" velocity="1" lower="0" upper="0" />
+    <limit effort="12" velocity="15" lower="0" upper="0" />
   </joint>
   <joint name="back_right_wheel_link_joint" type="continuous">
@@ -259,5 +259,5 @@
     <child link="back_right_wheel_link" />
     <axis xyz="0 1 0" />
-    <limit effort="10" velocity="1" lower="0" upper="0" />
+    <limit effort="12" velocity="15" lower="0" upper="0" />
   </joint>
   <joint name="chassis_link_joint" type="fixed">
@@ -271,12 +271,12 @@
     <child link="front_left_wheel_link" />
     <axis xyz="0 1 0" />
-    <limit effort="10" velocity="1" lower="0" upper="0" />
-  </joint>
-  <joint name="left_back_wheel_link_joint" type="continuous">
+    <limit effort="12" velocity="15" lower="0" upper="0" />
+  </joint>
+  <joint name="front_right_wheel_link_joint" type="continuous">
     <origin xyz="0.247131 -0.0135 -0.201737" rpy="0 0 0" />
     <parent link="right_bogie_link" />
-    <child link="left_back_wheel_link" />
-    <axis xyz="0 1 0" />
-    <limit effort="10" velocity="1" lower="0" upper="0" />
+    <child link="front_right_wheel_link" />
+    <axis xyz="0 1 0" />
+    <limit effort="12" velocity="15" lower="0" upper="0" />
   </joint>
   <joint name="left_bogie_link_joint" type="revolute">
@@ -299,5 +299,5 @@
     <child link="middle_left_wheel_link" />
     <axis xyz="0 1 0" />
-    <limit effort="10" velocity="1" lower="0" upper="0" />
+    <limit effort="12" velocity="15" lower="0" upper="0" />
   </joint>
   <joint name="middle_right_wheel_link_joint" type="continuous">
@@ -306,5 +306,5 @@
     <child link="middle_right_wheel_link" />
     <axis xyz="0 1 0" />
-    <limit effort="10" velocity="1" lower="0" upper="0" />
+    <limit effort="12" velocity="15" lower="0" upper="0" />
   </joint>
   <joint name="right_bogie_link_joint" type="revolute">

File: src/rover_description/urdf/rover_sim.urdf (robot description, URDF)
Before this commit: robot rover, 14 links, 13 joints
Links:
- removed link left_back_wheel_link
- added link front_right_wheel_link, mass 3; collision cylinder length=0.184024 radius=0.119695; visual mesh filename=package://rover_description/urdf/meshes/front_right_wheel_l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
Joints:
- removed joint left_back_wheel_link_joint
- added joint front_right_wheel_link_joint: type continuous, parent right_bogie_link, child front_right_wheel_link, origin xyz=0.247131 -0.0135 -0.201737 rpy=0 0 0, axis 0 1 0, limit lower=0 upper=0 effort=12 velocity=15
- joint back_left_wheel_link_joint: limit lower=0 upper=0 effort=10 velocity=1 -> lower=0 upper=0 effort=12 velocity=15
- joint back_right_wheel_link_joint: limit lower=0 upper=0 effort=10 velocity=1 -> lower=0 upper=0 effort=12 velocity=15
- joint front_left_wheel_link_joint: limit lower=0 upper=0 effort=10 velocity=1 -> lower=0 upper=0 effort=12 velocity=15
- joint left_bogie_link_joint: limit lower=-3.141593 upper=3.141593 effort=10 velocity=1 -> lower=-0.5236 upper=0.5236 effort=10 velocity=1
- joint middle_left_wheel_link_joint: limit lower=0 upper=0 effort=10 velocity=1 -> lower=0 upper=0 effort=12 velocity=15
- joint middle_right_wheel_link_joint: limit lower=0 upper=0 effort=10 velocity=1 -> lower=0 upper=0 effort=12 velocity=15
- joint right_bogie_link_joint: limit lower=-3.141593 upper=3.141593 effort=10 velocity=1 -> lower=-0.5236 upper=0.5236 effort=10 velocity=1

File: src/rover_description/urdf/rover_sim.xacro (robot description, xacro)
@@ -95,14 +95,14 @@
     </collision>
   </link>
-  <link name="left_back_wheel_link">
-    <inertial>
-      <origin rpy="1.570796 0 0" xyz="-0.000784 -0.092012 0.001876"/>
-      <mass value="3"/>
-      <inertia ixx="0.019211" ixy="0" ixz="0" iyy="0.019211" iyz="0" izz="0.02149"/>
-    </inertial>
-    <visual>
-      <origin rpy="1.570796 0 0" xyz="-0.000784 -0.092012 0.001876"/>
-      <geometry>
-        <mesh filename="package://rover_description/urdf/meshes/left_back_wheel_link_visual.obj"/>
+  <link name="front_right_wheel_link">
+    <inertial>
+      <origin rpy="1.570796 0 0" xyz="-0.000784 -0.092012 0.001876"/>
+      <mass value="3"/>
+      <inertia ixx="0.019211" ixy="0" ixz="0" iyy="0.019211" iyz="0" izz="0.02149"/>
+    </inertial>
+    <visual>
+      <origin rpy="1.570796 0 0" xyz="-0.000784 -0.092012 0.001876"/>
+      <geometry>
+        <mesh filename="package://rover_description/urdf/meshes/front_right_wheel_link_visual.obj"/>
       </geometry>
       <material name="off_black"/>
@@ -261,5 +261,5 @@
     <child link="back_left_wheel_link"/>
     <axis xyz="0 1 0"/>
-    <limit effort="10" lower="0" upper="0" velocity="1"/>
+    <limit effort="12" lower="0" upper="0" velocity="15"/>
     <dynamics damping="1.0" friction="1.5"/>
   </joint>
@@ -269,5 +269,5 @@
     <child link="back_right_wheel_link"/>
     <axis xyz="0 1 0"/>
-    <limit effort="10" lower="0" upper="0" velocity="1"/>
+    <limit effort="12" lower="0" upper="0" velocity="15"/>
     <dynamics damping="1.0" friction="1.5"/>
   </joint>
@@ -282,13 +282,13 @@
     <child link="front_left_wheel_link"/>
     <axis xyz="0 1 0"/>
-    <limit effort="10" lower="0" upper="0" velocity="1"/>
-    <dynamics damping="1.0" friction="1.5"/>
-  </joint>
-  <joint name="left_back_wheel_link_joint" type="continuous">
+    <limit effort="12" lower="0" upper="0" velocity="15"/>
+    <dynamics damping="1.0" friction="1.5"/>
+  </joint>
+  <joint name="front_right_wheel_link_joint" type="continuous">
     <origin rpy="0 0 0" xyz="0.247131 -0.0135 -0.201737"/>
     <parent link="right_bogie_link"/>
-    <child link="left_back_wheel_link"/>
-    <axis xyz="0 1 0"/>
-    <limit effort="10" lower="0" upper="0" velocity="1"/>
+    <child link="front_right_wheel_link"/>
+    <axis xyz="0 1 0"/>
+    <limit effort="12" lower="0" upper="0" velocity="15"/>
     <dynamics damping="1.0" friction="1.5"/>
   </joint>
@@ -298,5 +298,5 @@
     <child link="left_bogie_link"/>
     <axis xyz="0 1 0"/>
-    <limit effort="10" lower="-3.141593" upper="3.141593" velocity="1"/>
+    <limit effort="10" lower="-0.5236" upper="0.5236" velocity="1"/>
     <dynamics damping="0.3" friction="0.5"/>
   </joint>
@@ -307,5 +307,5 @@
     <axis xyz="0 1 0"/>
     <limit effort="10" lower="-1.570795" upper="1.570795" velocity="1"/>
-    <dynamics damping="0.5" friction="10.0"/>
+    <dynamics damping="0.5" friction="1000.0"/>
   </joint>
   <joint name="middle_left_wheel_link_joint" type="continuous">
@@ -314,5 +314,5 @@
     <child link="middle_left_wheel_link"/>
     <axis xyz="0 1 0"/>
-    <limit effort="10" lower="0" upper="0" velocity="1"/>
+    <limit effort="12" lower="0" upper="0" velocity="15"/>
     <dynamics damping="1.0" friction="1.5"/>
   </joint>
@@ -322,5 +322,5 @@
     <child link="middle_right_wheel_link"/>
     <axis xyz="0 1 0"/>
-    <limit effort="10" lower="0" upper="0" velocity="1"/>
+    <limit effort="12" lower="0" upper="0" velocity="15"/>
     <dynamics damping="1.0" friction="1.5"/>
   </joint>
@@ -330,5 +330,5 @@
     <child link="right_bogie_link"/>
     <axis xyz="0 1 0"/>
-    <limit effort="10" lower="-3.141593" upper="3.141593" velocity="1"/>
+    <limit effort="10" lower="-0.5236" upper="0.5236" velocity="1"/>
     <dynamics damping="0.3" friction="0.5"/>
   </joint>
@@ -339,5 +339,5 @@
     <axis xyz="0 1 0"/>
     <limit effort="10" lower="-3.141593" upper="3.141593" velocity="1"/>
-    <dynamics damping="0.5" friction="10.0"/>
+    <dynamics damping="0.5" friction="1000.0"/>
   </joint>
   <joint name="zed_camera_link_joint" type="fixed">
@@ -362,5 +362,5 @@
       <left_joint>middle_left_wheel_link_joint</left_joint>
       <left_joint>back_left_wheel_link_joint</left_joint>
-      <right_joint>left_back_wheel_link_joint</right_joint>
+      <right_joint>front_right_wheel_link_joint</right_joint>
       <right_joint>middle_right_wheel_link_joint</right_joint>
       <right_joint>back_right_wheel_link_joint</right_joint>
@@ -457,5 +457,5 @@
     <visual><material><ambient>0.15 0.15 0.15 1</ambient><diffuse>0.2 0.2 0.2 1</diffuse><specular>0.1 0.1 0.1 1</specular></material></visual>
   </gazebo>
-  <gazebo reference="left_back_wheel_link">
+  <gazebo reference="front_right_wheel_link">
     <visual><material><ambient>0.15 0.15 0.15 1</ambient><diffuse>0.2 0.2 0.2 1</diffuse><specular>0.1 0.1 0.1 1</specular></material></visual>
   </gazebo>
