Commit message: Terrain mapper, jade on the terrain course, new course, Humble builds
- rover_traversability (new): terrain_mapper builds a rover-centred height
  map from the ZED depth cloud (self-filter for the rover's own body) and
  publishes slope/step/roughness costs on /traversability/costmap;
  check_terrain_map.py compares a saved map with the generated terrain.
- Terrain course: small hill, crossable trench, rock garden, 1 m big hill;
  markers moved, their fallback positions written to
  config/terrain_markers.yaml (goal_generator marker_poses parameter).
- jade on the course: jade_terrain.xacro (sim-only settings and nav
  sensors) and jade_terrain.launch.py (arm stowed before driving).
  rover_raw.xacro: bogie limits +-30 deg, rocker_friction and chassis_zed
  settings; jade.xacro turns the chassis ZED off (it duplicated the arm's
  and made jade's URDF invalid); common_properties.xacro: wheel friction and
  DiffDrive topics as settings, defaults unchanged.
- movement.py: no pivoting while driving (inner wheels keep part of the
  forward speed); back-ups only reset the recovery count once past the
  first stall, so it reaches ABORTED instead of looping.
- Humble: rover_arm_hardware, real_arm_teleop_node and moveit_goal_node
  switch between the Jazzy and Humble APIs at compile time (tested in a
  ros:humble container).
- README updated for all of the above.

Co-Authored-By: Claude Opus 5.5 <noreply@anthropic.com>

File: src/jade_description/urdf/common_properties.xacro (robot description, xacro)
@@ -1,4 +1,8 @@
 <?xml version="1.0"?>
 <robot xmlns:xacro="http://www.ros.org/wiki/xacro">
+  <!-- Topics for DiffDrive's wheel odometry. jade_terrain.xacro moves them aside so a
+       ground-truth odometry plugin can own /odom and odom -> chassis_footprint. -->
+  <xacro:arg name="diff_drive_odom_topic" default="odom" />
+  <xacro:arg name="diff_drive_tf_topic" default="tf" />
   <!-- Shiny Aluminum Gazebo Macro -->
   <xacro:macro name="gazebo_shiny_aluminum" params="link_name">
@@ -74,6 +78,6 @@
       <!-- ROS / Gazebo Communication -->
       <topic>cmd_vel</topic>
-      <odom_topic>odom</odom_topic>
-      <tf_topic>tf</tf_topic>
+      <odom_topic>$(arg diff_drive_odom_topic)</odom_topic>
+      <tf_topic>$(arg diff_drive_tf_topic)</tf_topic>
       <frame_id>odom</frame_id>
       <child_frame_id>chassis_footprint</child_frame_id>
@@ -81,33 +85,37 @@
     </plugin>
   </gazebo>
+  <!-- Wheel friction. Defaults keep jade's tuning; jade_terrain.xacro declares these args
+       first (first declaration wins) to change them for the terrain sim. -->
+  <xacro:arg name="wheel_mu1" default="0.5" />
+  <xacro:arg name="wheel_mu2" default="0.05" />
   <!-- Apply to front_left, front_right, rear_left, and rear_right wheel links -->
   <gazebo reference="front_left_wheel_link">
-    <mu1>0.5</mu1>
-    <mu2>0.05</mu2> <!-- Low secondary friction allows lateral sliding when turning -->
+    <mu1>$(arg wheel_mu1)</mu1>
+    <mu2>$(arg wheel_mu2)</mu2> <!-- Low secondary friction allows lateral sliding when turning -->
     <fdir1>1 0 0</fdir1>
   </gazebo>
   <gazebo reference="front_right_wheel_link">
-    <mu1>0.5</mu1>
-    <mu2>0.05</mu2> <!-- Low secondary friction allows lateral sliding when turning -->
+    <mu1>$(arg wheel_mu1)</mu1>
+    <mu2>$(arg wheel_mu2)</mu2> <!-- Low secondary friction allows lateral sliding when turning -->
     <fdir1>1 0 0</fdir1>
   </gazebo>
   <gazebo reference="middle_left_wheel_link">
-    <mu1>0.5</mu1>
-    <mu2>0.05</mu2> <!-- Low secondary friction allows lateral sliding when turning -->
+    <mu1>$(arg wheel_mu1)</mu1>
+    <mu2>$(arg wheel_mu2)</mu2> <!-- Low secondary friction allows lateral sliding when turning -->
     <fdir1>1 0 0</fdir1>
   </gazebo>
   <gazebo reference="middle_right_wheel_link">
-    <mu1>0.5</mu1>
-    <mu2>0.05</mu2> <!-- Low secondary friction allows lateral sliding when turning -->
+    <mu1>$(arg wheel_mu1)</mu1>
+    <mu2>$(arg wheel_mu2)</mu2> <!-- Low secondary friction allows lateral sliding when turning -->
     <fdir1>1 0 0</fdir1>
   </gazebo>
   <gazebo reference="back_left_wheel_link">
-    <mu1>0.5</mu1>
-    <mu2>0.05</mu2> <!-- Low secondary friction allows lateral sliding when turning -->
+    <mu1>$(arg wheel_mu1)</mu1>
+    <mu2>$(arg wheel_mu2)</mu2> <!-- Low secondary friction allows lateral sliding when turning -->
     <fdir1>1 0 0</fdir1>
   </gazebo>
   <gazebo reference="back_right_wheel_link">
-    <mu1>0.5</mu1>
-    <mu2>0.05</mu2> <!-- Low secondary friction allows lateral sliding when turning -->
+    <mu1>$(arg wheel_mu1)</mu1>
+    <mu2>$(arg wheel_mu2)</mu2> <!-- Low secondary friction allows lateral sliding when turning -->
     <fdir1>1 0 0</fdir1>
   </gazebo>

File: src/jade_description/urdf/jade.xacro (robot description, xacro)
@@ -1,4 +1,7 @@
 <?xml version="1.0"?>
 <robot xmlns:xacro="http://www.ros.org/wiki/xacro" name="jade">
+  <!-- The arm brings its own ZED on the stand, so rover_raw's placeholder chassis ZED is
+       turned off (two zed_camera_link links make the URDF invalid). -->
+  <xacro:arg name="chassis_zed" default="false" />
   <!-- 1. Global properties & color macros MUST come first -->
   <xacro:include filename="$(find jade_description)/urdf/common_properties.xacro" />

File: src/rover_description/urdf/rover_raw.urdf (robot description, URDF)
Before this commit: robot rover_test_version, 13 links, 12 joints
Joints:
- joint left_bogie_link_joint: limit lower=-3.141593 upper=3.141593 effort=10 velocity=1 -> lower=-0.5236 upper=0.5236 effort=10 velocity=1
- joint right_bogie_link_joint: limit lower=-3.141593 upper=3.141593 effort=10 velocity=1 -> lower=-0.5236 upper=0.5236 effort=10 velocity=1

File: src/rover_description/urdf/rover_raw.xacro (robot description, xacro)
@@ -7,4 +7,13 @@
 -->
 <robot xmlns:xacro="http://ros.org/xacro" name="rover_test_version">
+  <!-- Settings that a including file can change by declaring the same xacro:arg before its
+       include (the first declaration wins), or on the xacro command line:
+         rocker_friction  joint friction on both rockers (N·m). 0 = free, as on the real rover.
+                          The terrain sim locks them with 1000: Gazebo's DART engine ignores
+                          the rocker differential, so free rockers let the chassis pitch ~45 deg.
+         chassis_zed      the placeholder ZED on the chassis. Off when the arm (with its own
+                          ZED on the stand) is mounted, e.g. jade.xacro. -->
+  <xacro:arg name="rocker_friction" default="0.0" />
+  <xacro:arg name="chassis_zed" default="true" />
   <!-- Links -->
   <link name="back_left_wheel_link">
@@ -223,4 +232,5 @@
     </collision>
   </link>
+  <xacro:if value="$(arg chassis_zed)">
   <link name="zed_camera_link">
     <!-- Geometry copied from rover_arm_raw.xacro's zed_camera_link (the
@@ -246,4 +256,5 @@
     </collision>
   </link>
+  </xacro:if>
   <!-- Joints -->
   <joint name="back_left_wheel_link_joint" type="continuous">
@@ -285,5 +296,5 @@
     <child link="left_bogie_link" />
     <axis xyz="0 1 0" />
-    <limit effort="10" velocity="1" lower="-3.141593" upper="3.141593" />
+    <limit effort="10" velocity="1" lower="-0.5236" upper="0.5236" />
   </joint>
   <joint name="left_rocker_link_joint" type="revolute">
@@ -293,4 +304,5 @@
     <axis xyz="0 1 0" />
     <limit effort="10" velocity="1" lower="-1.570795" upper="1.570795" />
+    <dynamics friction="$(arg rocker_friction)" />
   </joint>
   <joint name="middle_left_wheel_link_joint" type="continuous">
@@ -313,5 +325,5 @@
     <child link="right_bogie_link" />
     <axis xyz="0 1 0" />
-    <limit effort="10" velocity="1" lower="-3.141593" upper="3.141593" />
+    <limit effort="10" velocity="1" lower="-0.5236" upper="0.5236" />
   </joint>
   <joint name="right_rocker_link_joint" type="revolute">
@@ -321,5 +333,7 @@
     <axis xyz="0 1 0" />
     <limit effort="10" velocity="1" lower="-3.141593" upper="3.141593" />
-  </joint>
+    <dynamics friction="$(arg rocker_friction)" />
+  </joint>
+  <xacro:if value="$(arg chassis_zed)">
   <joint name="zed_camera_link_joint" type="fixed">
     <!-- TODO: PLACEHOLDER. chassis_link and the arm's stand_link have no
@@ -337,3 +351,4 @@
     <child link="zed_camera_link" />
   </joint>
+  </xacro:if>
 </robot>
