Commit message: Soft and hard joint limits; palm roll revolute +-90 deg with an RViz slider
The palm was a continuous joint (with a leftover lower=upper=0 limit), so
MoveIt loaded it unbounded and RViz's Joints tab gave it no editor at all.
It is now revolute, limited to +-90 deg (a safe range until the real one is
known).

Making it limited exposed a sim problem: in Gazebo (DART) a joint driven onto
its URDF limit stayed stuck there (reproduced on the palm and the wrist). So
all five arm joints now have:
- soft limits (the ranges the arm uses) in MoveIt's joint_limits.yaml and
  real_arm_teleop_node.cpp: base +-90, shoulder -90..+22.5, elbow +-180,
  wrist +-90, palm +-90 deg
- URDF hard stops 10 deg wider, so MoveIt never plans onto them

Also: the sim's palm command limit and jade's control.xacro match the new
range; README documents soft vs hard limits.

Tested in Gazebo (headless): every joint goes to its soft limit and back
(previously the palm and wrist froze at +-90). MoveIt plans palm goals of
+-95 deg to +-90 deg. The RViz Joints-tab palm slider works (checked by
hand). rover_sim's gz_ros2_control does not enforce the command min/max, so
trajectories published by hand can still reach the hard stops in sim.

Co-Authored-By: Claude Opus 5.5 <noreply@anthropic.com>

File: src/jade_description/urdf/control.xacro (robot description, xacro)
@@ -41,7 +41,10 @@
       <state_interface name="effort"/>
     </joint>
-    <!-- continuous joint (wrist roll) — no hard position limit -->
+    <!-- wrist roll: revolute, +-90 deg (rover_arm.xacro) -->
     <joint name="palm_link_joint">
-      <command_interface name="position"/>
+      <command_interface name="position">
+        <param name="min">-1.570796</param>
+        <param name="max">1.570796</param>
+      </command_interface>
       <state_interface name="position"/>
       <state_interface name="velocity"/>

File: src/rover_arm_description/urdf/rover_arm.xacro (robot description, xacro)
@@ -350,4 +350,11 @@
     </collision>
   </link>
+  <!-- Arm joint limits: the <limit> lower/upper below are HARD STOPS, 10 deg outside the
+       ranges the arm actually uses. The working (soft) limits are in
+       rover_arm_moveit_config/config/joint_limits.yaml (MoveIt, RViz sliders) and
+       real_arm_teleop_node.cpp. rover_arm_sim.xacro's command min/max match them, but
+       gz_ros2_control doesn't enforce those. In Gazebo's DART engine a velocity-driven joint
+       driven onto its stop could stay stuck there; the 10 deg margin keeps MoveIt's plans
+       clear of it. -->
   <!-- Joints. Arm efforts are the CAD motor torques (from the v1 export); 10 Nm everywhere
        was too weak to lift the arm in a physics engine that enforces effort limits. -->
@@ -357,5 +364,5 @@
     <child link="base_link" />
     <axis xyz="0 0 1" />
-    <limit effort="34.32" velocity="1" lower="-1.570795" upper="1.570795" />
+    <limit effort="34.32" velocity="1" lower="-1.745329" upper="1.745329" />
     <!-- friction was 75 Nm: more than the joint's 34 Nm effort, so under DART the base could
          never turn. The real base is held by its motor/gearbox, not by joint friction. -->
@@ -372,5 +379,5 @@
     <child link="elbow_link" />
     <axis xyz="0 1 0" />
-    <limit effort="123.56" velocity="1" lower="-3.141593" upper="3.141593" />
+    <limit effort="123.56" velocity="1" lower="-3.316126" upper="3.316126" />
   </joint>
   <joint name="left_finger_back_bottom_link_joint" type="revolute">
@@ -414,10 +421,13 @@
     <mimic joint="right_finger_back_top_link_joint" />
   </joint>
-  <joint name="palm_link_joint" type="continuous">
+  <joint name="palm_link_joint" type="revolute">
     <origin xyz="0.163045 -0.000975 0.000003" rpy="0 0 0" />
     <parent link="wrist_link" />
     <child link="palm_link" />
     <axis xyz="1 0 0" />
-    <limit effort="10" velocity="1" lower="0" upper="0" />
+    <!-- Palm roll limited to +-90 deg for now (safe range; set the real bevel/cable range
+         when known). Revolute rather than continuous: MoveIt ignores position limits on a
+         continuous joint, and RViz's Joints tab gives an unbounded joint no editor. -->
+    <limit effort="10" velocity="1" lower="-1.745329" upper="1.745329" />
   </joint>
   <joint name="right_finger_back_bottom_link_joint" type="revolute">
@@ -468,5 +478,5 @@
          export had upper="0": no motion below horizontal, and a joint starting exactly on its
          limit is frozen in Gazebo's DART engine. Confirm with the mechanical team. -->
-    <limit effort="137.3" velocity="1" lower="-1.570795" upper="0.3927" />
+    <limit effort="137.3" velocity="1" lower="-1.745329" upper="0.567232" />
   </joint>
   <joint name="wrist_link_joint" type="revolute">
@@ -475,5 +485,5 @@
     <child link="wrist_link" />
     <axis xyz="0 1 0" />
-    <limit effort="27.46" velocity="1" lower="-1.570795" upper="1.570795" />
+    <limit effort="27.46" velocity="1" lower="-1.745329" upper="1.745329" />
   </joint>
   <joint name="zed_camera_link_joint" type="fixed">

File: src/rover_arm_description/urdf/rover_arm_sim.xacro (robot description, xacro)
@@ -50,5 +50,5 @@
       <xacro:gz_joint name="elbow_link_joint" lower="-3.141593" upper="3.141593"/>
       <xacro:gz_joint name="wrist_link_joint" lower="-1.570795" upper="1.570795"/>
-      <xacro:gz_joint name="palm_link_joint" lower="-6.283185" upper="6.283185"/>
+      <xacro:gz_joint name="palm_link_joint" lower="-1.570796" upper="1.570796"/>  <!-- matches the URDF limit -->
       <!-- the gripper's one actuated joint -->
       <xacro:gz_joint name="right_finger_back_top_link_joint" lower="-0.785398" upper="0.523598"/>
